Commit message: Added proper velocity limits for safety

File: motion_controller_models/models/omx/omx_f.urdf (robot description, URDF)
Before this commit: robot omx_f, 10 links, 9 joints
Joints:
- joint gripper_joint_1: limit lower=-6.283185307179586 upper=6.283185307179586 effort=1000 velocity=4.8 -> lower=0 upper=1.74533 effort=1000 velocity=1.5
- joint gripper_joint_2: limit lower=-6.283185307179586 upper=6.283185307179586 effort=1000 velocity=4.8 -> lower=0 upper=1.74533 effort=1000 velocity=1.5
- joint joint1: limit lower=-6.283185307179586 upper=6.283185307179586 effort=1000 velocity=4.8 -> lower=-4.71239 upper=6.28319 effort=1000 velocity=1.5
- joint joint2: limit lower=-6.283185307179586 upper=6.283185307179586 effort=1000 velocity=4.8 -> lower=-2.0944 upper=1.5708 effort=1000 velocity=1.5
- joint joint3: limit lower=-6.283185307179586 upper=6.283185307179586 effort=1000 velocity=4.8 -> lower=-2.0944 upper=1.5708 effort=1000 velocity=1.5
- joint joint4: limit lower=-6.283185307179586 upper=6.283185307179586 effort=1000 velocity=4.8 -> lower=-1.74533 upper=1.74533 effort=1000 velocity=1.5
- joint joint5: limit lower=-6.283185307179586 upper=6.283185307179586 effort=1000 velocity=4.8 -> lower=-4.71239 upper=4.71239 effort=1000 velocity=1.5

File: motion_controller_models/models/omy/omy_3m.urdf (robot description, URDF)
Before this commit: robot omy_3m, 9 links, 8 joints
Joints:
- joint joint1: limit lower=-6.283185307179586 upper=6.283185307179586 effort=1000 velocity=4.8 -> lower=-6.283185307179586 upper=6.283185307179586 effort=1000 velocity=1.5
- joint joint2: limit lower=-6.283185307179586 upper=6.283185307179586 effort=1000 velocity=4.8 -> lower=-6.283185307179586 upper=6.283185307179586 effort=1000 velocity=1.5
- joint joint3: limit lower=-6.283185307179586 upper=6.283185307179586 effort=1000 velocity=4.8 -> lower=-2.61799 upper=2.61799 effort=1000 velocity=1.5
- joint joint4: limit lower=-6.283185307179586 upper=6.283185307179586 effort=1000 velocity=4.8 -> lower=-6.283185307179586 upper=6.283185307179586 effort=1000 velocity=1.5
- joint joint5: limit lower=-6.283185307179586 upper=6.283185307179586 effort=1000 velocity=4.8 -> lower=-6.283185307179586 upper=6.283185307179586 effort=1000 velocity=1.5
- joint joint6: limit lower=-6.283185307179586 upper=6.283185307179586 effort=1000 velocity=4.8 -> lower=-6.283185307179586 upper=6.283185307179586 effort=1000 velocity=1.5

File: motion_controller_models/models/omy/omy_f3m.urdf (robot description, URDF)
Before this commit: robot omy_f3m, 15 links, 14 joints
Joints:
- joint joint1: limit lower=-6.283185307179586 upper=6.283185307179586 effort=1000 velocity=4.8 -> lower=-6.283185307179586 upper=6.283185307179586 effort=1000 velocity=1.5
- joint joint2: limit lower=-6.283185307179586 upper=6.283185307179586 effort=1000 velocity=4.8 -> lower=-6.283185307179586 upper=6.283185307179586 effort=1000 velocity=1.5
- joint joint3: limit lower=-6.283185307179586 upper=6.283185307179586 effort=1000 velocity=4.8 -> lower=-2.61799 upper=2.61799 effort=1000 velocity=1.5
- joint joint4: limit lower=-6.283185307179586 upper=6.283185307179586 effort=1000 velocity=4.8 -> lower=-6.283185307179586 upper=6.283185307179586 effort=1000 velocity=1.5
- joint joint5: limit lower=-6.283185307179586 upper=6.283185307179586 effort=1000 velocity=4.8 -> lower=-6.283185307179586 upper=6.283185307179586 effort=1000 velocity=1.5
- joint joint6: limit lower=-6.283185307179586 upper=6.283185307179586 effort=1000 velocity=4.8 -> lower=-6.283185307179586 upper=6.283185307179586 effort=1000 velocity=1.5
