Commit message: Add omy leader impedance controller for testing torque interface

File: cyclo_motion_controller_models/models/omy/omy_l100.urdf (robot description, URDF)
Before this commit: robot omy_l100, 9 links, 8 joints
Links:
- link link0: geometry visual mesh filename=package://open_manipulator_description/meshes/omy_l100/base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 scale=0.001 0.001 0.001
- link link1: geometry visual mesh filename=package://open_manipulator_description/meshes/omy_l100/link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 scale=0.001 0.001 0.001
- link link2: geometry visual mesh filename=package://open_manipulator_description/meshes/omy_l100/link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 scale=0.001 0.001 0.001
- link link3: geometry visual mesh filename=package://open_manipulator_description/meshes/omy_l100/link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 scale=0.001 0.001 0.001
- link link4: geometry visual mesh filename=package://open_manipulator_description/meshes/omy_l100/link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 scale=0.001 0.001 0.001
- link link5: geometry visual mesh filename=package://open_manipulator_description/meshes/omy_l100/link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 scale=0.001 0.001 0.001
- link link6: geometry visual mesh filename=package://open_manipulator_description/meshes/omy_l100/link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 scale=0.001 0.001 0.001
- link link7: geometry visual mesh filename=package://open_manipulator_description/meshes/omy_l100/link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 scale=0.001 0.001 0.001
