Commit message: Fixed joint7 position limits

File: cyclo_motion_controller_models/models/ai_worker/ffw_sg2_follower.urdf (robot description, URDF)
Before this commit: robot ffw_sg2_follower, 42 links, 41 joints
Joints:
- joint arm_l_joint7: limit lower=-1.8201 upper=1.5804 effort=1000 velocity=4.8 -> lower=-1.5804 upper=1.8201 effort=1000 velocity=4.8
- joint arm_r_joint7: limit lower=-1.5804 upper=1.8201 effort=1000 velocity=4.8 -> lower=-1.8201 upper=1.5804 effort=1000 velocity=4.8
