Commit message: Modified gripper collision spheres and srdfs

File: cyclo_motion_controller_models/models/ai_worker/ffw_bg2_follower.urdf (robot description, URDF)
Before this commit: robot ffw_bg2_follower, 35 links, 34 joints
Links:
- link arm_l_link7: geometry collision box size=0.023 0.042 0.042; collision cylinder length=0.06 radius=0.085
- link arm_r_link7: geometry collision box size=0.023 0.042 0.042; collision cylinder length=0.06 radius=0.085
- link gripper_l_rh_p12_rn_base: geometry collision sphere radius=0.085; visual mesh filename=package://ffw_description/meshes/common/rh_p12_rn_a/base.stl scale=0.001 0.001 0.001
- link gripper_r_rh_p12_rn_base: geometry collision sphere radius=0.085; visual mesh filename=package://ffw_description/meshes/common/rh_p12_rn_a/base.stl scale=0.001 0.001 0.001

File: cyclo_motion_controller_models/models/ai_worker/ffw_bh5_follower.urdf (robot description, URDF)
Before this commit: robot ffw_bh5_follower, 18 links, 17 joints
Links:
- link arm_l_link7: geometry collision box size=0.023 0.042 0.042; collision cylinder length=0.06 radius=0.085
- link arm_r_link7: geometry collision box size=0.023 0.042 0.042; collision cylinder length=0.06 radius=0.085
- link hx5_d20_left_base: geometry collision sphere radius=0.089; collision sphere radius=0.095
- link hx5_d20_right_base: geometry collision sphere radius=0.089; collision sphere radius=0.095

File: cyclo_motion_controller_models/models/ai_worker/ffw_f1_follower.urdf (robot description, URDF)
Before this commit: robot ffw_f1_follower, 20 links, 19 joints
Links:
- added link gripper_l_hx2_d1_base; collision sphere radius=0.085
- added link gripper_r_hx2_d1_base; collision sphere radius=0.085
- link arm_l_link7: geometry collision box size=0.049953 0.037432 0.077001; collision cylinder length=0.04 radius=0.085
- link arm_r_link7: geometry collision box size=0.049953 0.037432 0.077001; collision cylinder length=0.04 radius=0.085
Joints:
- added joint gripper_l_joint: type fixed, parent arm_l_link7, child gripper_l_hx2_d1_base, origin xyz=0.00025 0 -0.05 rpy=3.14159265358979 0 0
- added joint gripper_r_joint: type fixed, parent arm_r_link7, child gripper_r_hx2_d1_base, origin xyz=0.00025 0 -0.05 rpy=3.14159265358979 0 0

File: cyclo_motion_controller_models/models/ai_worker/ffw_f2_follower.urdf (robot description, URDF)
Before this commit: robot ffw_f2_follower, 20 links, 19 joints
Links:
- added link gripper_l_hx2_d1_base; collision sphere radius=0.085
- added link gripper_r_hx2_d1_base; collision sphere radius=0.085
- link arm_l_link7: geometry collision box size=0.049953 0.037432 0.077001; collision cylinder length=0.04 radius=0.085
- link arm_r_link7: geometry collision box size=0.049953 0.037432 0.077001; collision cylinder length=0.04 radius=0.085
Joints:
- added joint gripper_l_joint: type fixed, parent arm_l_link7, child gripper_l_hx2_d1_base, origin xyz=0.00025 0 -0.05 rpy=3.14159265358979 0 0
- added joint gripper_r_joint: type fixed, parent arm_r_link7, child gripper_r_hx2_d1_base, origin xyz=0.00025 0 -0.05 rpy=3.14159265358979 0 0

File: cyclo_motion_controller_models/models/ai_worker/ffw_sg2_follower.urdf (robot description, URDF)
Before this commit: robot ffw_sg2_follower, 42 links, 41 joints
Links:
- link arm_l_link7: geometry collision box size=0.023 0.042 0.042; collision cylinder length=0.06 radius=0.085
- link arm_r_link7: geometry collision box size=0.023 0.042 0.042; collision cylinder length=0.06 radius=0.085
- link gripper_l_rh_p12_rn_base: geometry collision sphere radius=0.085; visual mesh filename=package://ffw_description/meshes/common/rh_p12_rn_a/base.stl scale=0.001 0.001 0.001
- link gripper_r_rh_p12_rn_base: geometry collision sphere radius=0.085; visual mesh filename=package://ffw_description/meshes/common/rh_p12_rn_a/base.stl scale=0.001 0.001 0.001

File: cyclo_motion_controller_models/models/ai_worker/ffw_sh5_follower.urdf (robot description, URDF)
Before this commit: robot ffw_sh5_follower, 18 links, 17 joints
Links:
- link arm_l_link7: geometry collision box size=0.023 0.042 0.042; collision cylinder length=0.06 radius=0.085
- link arm_r_link7: geometry collision box size=0.023 0.042 0.042; collision cylinder length=0.06 radius=0.085
- link hx5_d20_left_base: geometry collision sphere radius=0.089; collision sphere radius=0.095
- link hx5_d20_right_base: geometry collision sphere radius=0.089; collision sphere radius=0.095
