Commit message: Modified sh5 urdf and added sh5 urdf view launch

File: cyclo_motion_controller_models/models/ai_worker/ffw_sh5_follower.urdf (robot description, URDF)
Before this commit: robot ffw_sh5_follower, 18 links, 17 joints
Links:
- added link camera_left_bottom_screw_frame
- added link camera_left_link; visual mesh filename=package://realsense2_description/meshes/d405.stl scale=0.001 0.001 0.001
- added link camera_right_bottom_screw_frame
- added link camera_right_link; visual mesh filename=package://realsense2_description/meshes/d405.stl scale=0.001 0.001 0.001
- added link finger_end_l_link1; visual box size=0.01 0.01 0.01
- added link finger_end_l_link2; visual box size=0.01 0.01 0.01
- added link finger_end_l_link3; visual box size=0.01 0.01 0.01
- added link finger_end_l_link4; visual box size=0.01 0.01 0.01
- added link finger_end_l_link5; visual box size=0.01 0.01 0.01
- added link finger_end_r_link1; visual box size=0.01 0.01 0.01
- added link finger_end_r_link2; visual box size=0.01 0.01 0.01
- added link finger_end_r_link3; visual box size=0.01 0.01 0.01
- added link finger_end_r_link4; visual box size=0.01 0.01 0.01
- added link finger_end_r_link5; visual box size=0.01 0.01 0.01
- added link finger_l_link1; visual mesh filename=package://ffw_description/meshes/common/hx5_d20/hx5_d20_lef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 scale=0.001 0.001 0.001
- added link finger_l_link10; visual mesh filename=package://ffw_description/meshes/common/hx5_d20/hx5_d20_lef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 scale=0.001 0.001 0.001
- added link finger_l_link11; visual mesh filename=package://ffw_description/meshes/common/hx5_d20/hx5_d20_lef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 scale=0.001 0.001 0.001
- added link finger_l_link12; visual mesh filename=package://ffw_description/meshes/common/hx5_d20/hx5_d20_lef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 scale=0.001 0.001 0.001
- added link finger_l_link13; visual mesh filename=package://ffw_description/meshes/common/hx5_d20/hx5_d20_lef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 scale=0.001 0.001 0.001
- added link finger_l_link14; visual mesh filename=package://ffw_description/meshes/common/hx5_d20/hx5_d20_lef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 scale=0.001 0.001 0.001
- added link finger_l_link15; visual mesh filename=package://ffw_description/meshes/common/hx5_d20/hx5_d20_lef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 scale=0.001 0.001 0.001
- added link finger_l_link16; visual mesh filename=package://ffw_description/meshes/common/hx5_d20/hx5_d20_lef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 scale=0.001 0.001 0.001
- added link finger_l_link17; visual mesh filename=package://ffw_description/meshes/common/hx5_d20/hx5_d20_lef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 scale=0.001 0.001 0.001
- added link finger_l_link18; visual mesh filename=package://ffw_description/meshes/common/hx5_d20/hx5_d20_lef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 scale=0.001 0.001 0.001
- added link finger_l_link19; visual mesh filename=package://ffw_description/meshes/common/hx5_d20/hx5_d20_lef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 scale=0.001 0.001 0.001
- added link finger_l_link2; visual mesh filename=package://ffw_description/meshes/common/hx5_d20/hx5_d20_lef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 scale=0.001 0.001 0.001
- added link finger_l_link20; visual mesh filename=package://ffw_description/meshes/common/hx5_d20/hx5_d20_lef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 scale=0.001 0.001 0.001
- added link finger_l_link3; visual mesh filename=package://ffw_description/meshes/common/hx5_d20/hx5_d20_lef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 scale=0.001 0.001 0.001
- added link finger_l_link4; visual mesh filename=package://ffw_description/meshes/common/hx5_d20/hx5_d20_lef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 scale=0.001 0.001 0.001
- added link finger_l_link5; visual mesh filename=package://ffw_description/meshes/common/hx5_d20/hx5_d20_lef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 scale=0.001 0.001 0.001
- added link finger_l_link6; visual mesh filename=package://ffw_description/meshes/common/hx5_d20/hx5_d20_lef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 scale=0.001 0.001 0.001
- added link finger_l_link7; visual mesh filename=package://ffw_description/meshes/common/hx5_d20/hx5_d20_lef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 scale=0.001 0.001 0.001
- added link finger_l_link8; visual mesh filename=package://ffw_description/meshes/common/hx5_d20/hx5_d20_lef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 scale=0.001 0.001 0.001
- added link finger_l_link9; visual mesh filename=package://ffw_description/meshes/common/hx5_d20/hx5_d20_lef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 scale=0.001 0.001 0.001
- added link finger_r_link1; visual mesh filename=package://ffw_description/meshes/common/hx5_d20/hx5_d20_rig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 scale=0.001 0.001 0.001
- added link finger_r_link10; visual mesh filename=package://ffw_description/meshes/common/hx5_d20/hx5_d20_rig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 scale=0.001 0.001 0.001
- added link finger_r_link11; visual mesh filename=package://ffw_description/meshes/common/hx5_d20/hx5_d20_rig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 scale=0.001 0.001 0.001
- added link finger_r_link12; visual mesh filename=package://ffw_description/meshes/common/hx5_d20/hx5_d20_rig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 scale=0.001 0.001 0.001
- added link finger_r_link13; visual mesh filename=package://ffw_description/meshes/common/hx5_d20/hx5_d20_rig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 scale=0.001 0.001 0.001
- added link finger_r_link14; visual mesh filename=package://ffw_description/meshes/common/hx5_d20/hx5_d20_rig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 scale=0.001 0.001 0.001
- added link finger_r_link15; visual mesh filename=package://ffw_description/meshes/common/hx5_d20/hx5_d20_rig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 scale=0.001 0.001 0.001
- added link finger_r_link16; visual mesh filename=package://ffw_description/meshes/common/hx5_d20/hx5_d20_rig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 scale=0.001 0.001 0.001
- added link finger_r_link17; visual mesh filename=package://ffw_description/meshes/common/hx5_d20/hx5_d20_rig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 scale=0.001 0.001 0.001
- added link finger_r_link18; visual mesh filename=package://ffw_description/meshes/common/hx5_d20/hx5_d20_rig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 scale=0.001 0.001 0.001
- added link finger_r_link19; visual mesh filename=package://ffw_description/meshes/common/hx5_d20/hx5_d20_rig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 scale=0.001 0.001 0.001
- added link finger_r_link2; visual mesh filename=package://ffw_description/meshes/common/hx5_d20/hx5_d20_rig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 scale=0.001 0.001 0.001
- added link finger_r_link20; visual mesh filename=package://ffw_description/meshes/common/hx5_d20/hx5_d20_rig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 scale=0.001 0.001 0.001
- added link finger_r_link3; visual mesh filename=package://ffw_description/meshes/common/hx5_d20/hx5_d20_rig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 scale=0.001 0.001 0.001
- added link finger_r_link4; visual mesh filename=package://ffw_description/meshes/common/hx5_d20/hx5_d20_rig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 scale=0.001 0.001 0.001
- added link finger_r_link5; visual mesh filename=package://ffw_description/meshes/common/hx5_d20/hx5_d20_rig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 scale=0.001 0.001 0.001
- added link finger_r_link6; visual mesh filename=package://ffw_description/meshes/common/hx5_d20/hx5_d20_rig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 scale=0.001 0.001 0.001
- added link finger_r_link7; visual mesh filename=package://ffw_description/meshes/common/hx5_d20/hx5_d20_rig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 scale=0.001 0.001 0.001
- added link finger_r_link8; visual mesh filename=package://ffw_description/meshes/common/hx5_d20/hx5_d20_rig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 scale=0.001 0.001 0.001
- added link finger_r_link9; visual mesh filename=package://ffw_description/meshes/common/hx5_d20/hx5_d20_rig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 scale=0.001 0.001 0.001
- added link head_link1; visual mesh filename=package://ffw_description/meshes/common/follower/ffw/head_l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 scale=0.001 0.001 0.001
- added link head_link2; collision sphere radius=0.1; visual mesh filename=package://ffw_description/meshes/common/follower/ffw/head_l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 scale=0.001 0.001 0.001
- added link imu_link
- added link left_wheel_drive_link; visual mesh filename=package://ffw_description/meshes/common/follower/ffw_swerve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 scale=0.001 0.001 0.001
- added link left_wheel_steer_link; visual mesh filename=package://ffw_description/meshes/common/follower/ffw_swerve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 scale=0.001 0.001 0.001
- added link lidar_l_link; visual cylinder length=0.03 radius=0.03
- added link lidar_r_link; visual cylinder length=0.03 radius=0.03
- added link lift_link; visual mesh filename=package://ffw_description/meshes/common/follower/ffw_swerve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 scale=0.001 0.001 0.001
- added link rear_wheel_drive_link; visual mesh filename=package://ffw_description/meshes/common/follower/ffw_swerve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 scale=0.001 0.001 0.001
- added link rear_wheel_steer_link; visual mesh filename=package://ffw_description/meshes/common/follower/ffw_swerve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 scale=0.001 0.001 0.001
- added link right_wheel_drive_link; visual mesh filename=package://ffw_description/meshes/common/follower/ffw_swerve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 scale=0.001 0.001 0.001
- added link right_wheel_steer_link; visual mesh filename=package://ffw_description/meshes/common/follower/ffw_swerve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 scale=0.001 0.001 0.001
- added link world
- added link zed_camera_center; visual mesh filename=package://ffw_description/meshes/common/follower/zedm.stl scale=0.001 0.001 0.001
- added link zed_camera_link
- added link zed_left_camera_frame
- added link zed_left_camera_optical_frame
- added link zed_right_camera_frame
- added link zed_right_camera_optical_frame
- link arm_base_link: geometry collision box size=0.2 0.1 0.63; collision box size=0.2 0.1 0.63
- link arm_l_link1: geometry visual mesh filename=package://ffw_description/meshes/common/follower/ffw/arm_l_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 scale=0.001 0.001 0.001
- link arm_l_link2: geometry collision cylinder length=0.30 radius=0.07; collision sphere radius=0.07
- link arm_l_link3: geometry visual mesh filename=package://ffw_description/meshes/common/follower/ffw/arm_l_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 scale=0.001 0.001 0.001
- link arm_l_link4: geometry collision cylinder length=0.3 radius=0.07; collision sphere radius=0.07
- link arm_l_link5: geometry visual mesh filename=package://ffw_description/meshes/common/follower/ffw/arm_l_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 scale=0.001 0.001 0.001
- link arm_l_link6: geometry visual mesh filename=package://ffw_description/meshes/common/follower/ffw/arm_l_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 scale=0.001 0.001 0.001
- link arm_l_link7: geometry collision box size=0.023 0.042 0.042; collision cylinder length=0.06 radius=0.085
- link arm_r_link1: geometry visual mesh filename=package://ffw_description/meshes/common/follower/ffw/arm_r_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 scale=0.001 0.001 0.001
- link arm_r_link2: geometry collision cylinder length=0.30 radius=0.07; collision sphere radius=0.07
- link arm_r_link3: geometry visual mesh filename=package://ffw_description/meshes/common/follower/ffw/arm_r_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 scale=0.001 0.001 0.001
- link arm_r_link4: geometry collision cylinder length=0.3 radius=0.07; collision sphere radius=0.07
- link arm_r_link5: geometry visual mesh filename=package://ffw_description/meshes/common/follower/ffw/arm_r_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 scale=0.001 0.001 0.001
- link arm_r_link6: geometry visual mesh filename=package://ffw_description/meshes/common/follower/ffw/arm_r_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 scale=0.001 0.001 0.001
- link arm_r_link7: geometry collision box size=0.023 0.042 0.042; collision cylinder length=0.06 radius=0.085
- link base_link: geometry collision box size=0.6 0.4 0.3; collision cylinder length=0.4 radius=0.15
- link hx5_d20_left_base: geometry collision box size=0.06093245 0.11672498 0.24903000; visual mesh filename=package://ffw_description/meshes/common/hx5_d20/hx5_d20_lef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 scale=0.001 0.001 0.001
- link hx5_d20_right_base: geometry collision box size=0.06092238 0.11672498 0.24903000; visual mesh filename=package://ffw_description/meshes/common/hx5_d20/hx5_d20_rig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 scale=0.001 0.001 0.001
Joints:
- added joint camera_left_joint: type fixed, parent arm_l_link7, child camera_left_bottom_screw_frame, origin xyz=0.108236 -0.021 -0.062552 rpy=-1.57079632679 1.66678943569 0
- added joint camera_left_link_joint: type fixed, parent camera_left_bottom_screw_frame, child camera_left_link, origin xyz=0.01085 0.009 0.021 rpy=0 0 0
- added joint camera_right_joint: type fixed, parent arm_r_link7, child camera_right_bottom_screw_frame, origin xyz=0.108236 -0.021 -0.062552 rpy=-1.57079632679 1.66678943569 0
- added joint camera_right_link_joint: type fixed, parent camera_right_bottom_screw_frame, child camera_right_link, origin xyz=0.01085 0.009 0.021 rpy=0 0 0
- added joint finger_end_l_joint1: type fixed, parent finger_l_link4, child finger_end_l_link1, origin xyz=0.0 -0.03975 0.0 rpy=0 0 0
- added joint finger_end_l_joint2: type fixed, parent finger_l_link8, child finger_end_l_link2, origin xyz=0.0 0.0 0.02425 rpy=0 0 0
- added joint finger_end_l_joint3: type fixed, parent finger_l_link12, child finger_end_l_link3, origin xyz=0.0 0.0 0.02425 rpy=0 0 0
- added joint finger_end_l_joint4: type fixed, parent finger_l_link16, child finger_end_l_link4, origin xyz=0.0 0.0 0.02425 rpy=0 0 0
- added joint finger_end_l_joint5: type fixed, parent finger_l_link20, child finger_end_l_link5, origin xyz=0.0 0.0 0.02425 rpy=0 0 0
- added joint finger_end_r_joint1: type fixed, parent finger_r_link4, child finger_end_r_link1, origin xyz=0.0 0.03975 0.0 rpy=0 0 0
- added joint finger_end_r_joint2: type fixed, parent finger_r_link8, child finger_end_r_link2, origin xyz=0.0 0.0 0.02425 rpy=0 0 0
- added joint finger_end_r_joint3: type fixed, parent finger_r_link12, child finger_end_r_link3, origin xyz=0.0 0.0 0.02425 rpy=0 0 0
- added joint finger_end_r_joint4: type fixed, parent finger_r_link16, child finger_end_r_link4, origin xyz=0.0 0.0 0.02425 rpy=0 0 0
- added joint finger_end_r_joint5: type fixed, parent finger_r_link20, child finger_end_r_link5, origin xyz=0.0 0.0 0.02425 rpy=0 0 0
- added joint finger_l_joint1: type fixed, parent hx5_d20_left_base, child finger_l_link1, origin xyz=-0.0125 -0.03493 0.04475 rpy=0 0 0
- added joint finger_l_joint10: type fixed, parent finger_l_link9, child finger_l_link10, origin xyz=0.0165 0.0 0.0235 rpy=0 0 0
- added joint finger_l_joint11: type fixed, parent finger_l_link10, child finger_l_link11, origin xyz=0.0 0.0 0.0355 rpy=0 0 0
- added joint finger_l_joint12: type fixed, parent finger_l_link11, child finger_l_link12, origin xyz=0.0 0.0 0.0355 rpy=0 0 0
- added joint finger_l_joint13: type fixed, parent hx5_d20_left_base, child finger_l_link13, origin xyz=-0.0015 0.01792 0.10475 rpy=0 0 0
- added joint finger_l_joint14: type fixed, parent finger_l_link13, child finger_l_link14, origin xyz=0.0165 0.0 0.0235 rpy=0 0 0
- added joint finger_l_joint15: type fixed, parent finger_l_link14, child finger_l_link15, origin xyz=0.0 0.0 0.0355 rpy=0 0 0
- added joint finger_l_joint16: type fixed, parent finger_l_link15, child finger_l_link16, origin xyz=0.0 0.0 0.0355 rpy=0 0 0
- added joint finger_l_joint17: type fixed, parent hx5_d20_left_base, child finger_l_link17, origin xyz=-0.0015 0.04492 0.08575 rpy=0 0 0
- added joint finger_l_joint18: type fixed, parent finger_l_link17, child finger_l_link18, origin xyz=0.0165 0.0 0.0235 rpy=0 0 0
- added joint finger_l_joint19: type fixed, parent finger_l_link18, child finger_l_link19, origin xyz=0.0 0.0 0.0355 rpy=0 0 0
- added joint finger_l_joint2: type fixed, parent finger_l_link1, child finger_l_link2, origin xyz=0.039 0.0 0.0 rpy=0 0 0
- added joint finger_l_joint20: type fixed, parent finger_l_link19, child finger_l_link20, origin xyz=0.0 0.0 0.0355 rpy=0 0 0
- added joint finger_l_joint3: type fixed, parent finger_l_link2, child finger_l_link3, origin xyz=0.0 -0.028 0.0 rpy=0 0 0
- added joint finger_l_joint4: type fixed, parent finger_l_link3, child finger_l_link4, origin xyz=0.0 -0.0355 0.0 rpy=0 0 0
- added joint finger_l_joint5: type fixed, parent hx5_d20_left_base, child finger_l_link5, origin xyz=-0.0015 -0.03608 0.10275 rpy=0 0 0
- added joint finger_l_joint6: type fixed, parent finger_l_link5, child finger_l_link6, origin xyz=0.0165 0.0 0.0235 rpy=0 0 0
- added joint finger_l_joint7: type fixed, parent finger_l_link6, child finger_l_link7, origin xyz=0.0 0.0 0.0355 rpy=0 0 0
- added joint finger_l_joint8: type fixed, parent finger_l_link7, child finger_l_link8, origin xyz=0.0 0.0 0.0355 rpy=0 0 0
- added joint finger_l_joint9: type fixed, parent hx5_d20_left_base, child finger_l_link9, origin xyz=-0.0015 -0.00908 0.11053 rpy=0 0 0
- added joint finger_r_joint1: type fixed, parent hx5_d20_right_base, child finger_r_link1, origin xyz=-0.0125 0.03493 0.04475 rpy=0 0 0
- added joint finger_r_joint10: type fixed, parent finger_r_link9, child finger_r_link10, origin xyz=0.0165 0.0 0.0235 rpy=0 0 0
- added joint finger_r_joint11: type fixed, parent finger_r_link10, child finger_r_link11, origin xyz=0.0 0.0 0.0355 rpy=0 0 0
- added joint finger_r_joint12: type fixed, parent finger_r_link11, child finger_r_link12, origin xyz=0.0 0.0 0.0355 rpy=0 0 0
- added joint finger_r_joint13: type fixed, parent hx5_d20_right_base, child finger_r_link13, origin xyz=-0.0015 -0.01792 0.10475 rpy=0 0 0
- added joint finger_r_joint14: type fixed, parent finger_r_link13, child finger_r_link14, origin xyz=0.0165 0.0 0.0235 rpy=0 0 0
- added joint finger_r_joint15: type fixed, parent finger_r_link14, child finger_r_link15, origin xyz=0.0 0.0 0.0355 rpy=0 0 0
- added joint finger_r_joint16: type fixed, parent finger_r_link15, child finger_r_link16, origin xyz=0.0 0.0 0.0355 rpy=0 0 0
- added joint finger_r_joint17: type fixed, parent hx5_d20_right_base, child finger_r_link17, origin xyz=-0.0015 -0.04492 0.08575 rpy=0 0 0
- added joint finger_r_joint18: type fixed, parent finger_r_link17, child finger_r_link18, origin xyz=0.0165 0.0 0.0235 rpy=0 0 0
- added joint finger_r_joint19: type fixed, parent finger_r_link18, child finger_r_link19, origin xyz=0.0 0.0 0.0355 rpy=0 0 0
- added joint finger_r_joint2: type fixed, parent finger_r_link1, child finger_r_link2, origin xyz=0.039 0.0 0.0 rpy=0 0 0
- added joint finger_r_joint20: type fixed, parent finger_r_link19, child finger_r_link20, origin xyz=0.0 0.0 0.0355 rpy=0 0 0
- added joint finger_r_joint3: type fixed, parent finger_r_link2, child finger_r_link3, origin xyz=0.0 0.028 0.0 rpy=0 0 0
- added joint finger_r_joint4: type fixed, parent finger_r_link3, child finger_r_link4, origin xyz=0.0 0.0355 0.0 rpy=0 0 0
- added joint finger_r_joint5: type fixed, parent hx5_d20_right_base, child finger_r_link5, origin xyz=-0.0015 0.03608 0.10275 rpy=0 0 0
- added joint finger_r_joint6: type fixed, parent finger_r_link5, child finger_r_link6, origin xyz=0.0165 0.0 0.0235 rpy=0 0 0
- added joint finger_r_joint7: type fixed, parent finger_r_link6, child finger_r_link7, origin xyz=0.0 0.0 0.0355 rpy=0 0 0
- added joint finger_r_joint8: type fixed, parent finger_r_link7, child finger_r_link8, origin xyz=0.0 0.0 0.0355 rpy=0 0 0
- added joint finger_r_joint9: type fixed, parent hx5_d20_right_base, child finger_r_link9, origin xyz=-0.0015 0.00908 0.11053 rpy=0 0 0
- added joint head_joint1: type fixed, parent arm_base_link, child head_link1, origin xyz=0.049483 0 0.102130 rpy=0 0 0
- added joint head_joint2: type fixed, parent head_link1, child head_link2, origin xyz=0.040 0 0.054 rpy=0 0 0
- added joint imu_joint: type fixed, parent base_link, child imu_link, origin xyz=-0.1464 0.0 0.26 rpy=0 0 0
- added joint left_wheel_drive: type fixed, parent left_wheel_steer_link, child left_wheel_drive_link, origin xyz=0 0 -0.18905 rpy=0 0 0
- added joint left_wheel_steer: type fixed, parent base_link, child left_wheel_steer_link, origin xyz=0.1371 0.2554 0.27555 rpy=0 0 0
- added joint lidar_l_joint: type fixed, parent base_link, child lidar_l_link, origin xyz=-0.111881 0.240 0.34432 rpy=0 0 1.57079632679
- added joint lidar_r_joint: type fixed, parent base_link, child lidar_r_link, origin xyz=-0.111881 -0.240 0.34432 rpy=0 0 -1.57079632679
- added joint lift_fixed_joint: type fixed, parent base_link, child lift_link, origin xyz=0.0 0.0 0.0 rpy=0 0 0
- added joint rear_wheel_drive: type fixed, parent rear_wheel_steer_link, child rear_wheel_drive_link, origin xyz=0 0 -0.18905 rpy=0 0 0
- added joint rear_wheel_steer: type fixed, parent base_link, child rear_wheel_steer_link, origin xyz=-0.2899 0 0.27555 rpy=0 0 0
- added joint right_wheel_drive: type fixed, parent right_wheel_steer_link, child right_wheel_drive_link, origin xyz=0 0 -0.18905 rpy=0 0 0
- added joint right_wheel_steer: type fixed, parent base_link, child right_wheel_steer_link, origin xyz=0.1371 -0.2554 0.27555 rpy=0 0 0
- added joint world_fixed: type fixed, parent world, child base_link
- added joint zed_camera_center_joint: type fixed, parent zed_camera_link, child zed_camera_center, origin xyz=0 0 0.01325 rpy=0 0 0
- added joint zed_joint: type fixed, parent head_link2, child zed_camera_link, origin xyz=0.0238122 -0.00651797 -0.0242094 rpy=0 0 0
- added joint zed_left_camera_joint: type fixed, parent zed_camera_center, child zed_left_camera_frame, origin xyz=0 0.0315 0 rpy=0 0 0
- added joint zed_left_camera_optical_joint: type fixed, parent zed_left_camera_frame, child zed_left_camera_optical_frame, origin xyz=0 0 0 rpy=-1.57079632679 0.0 -1.57079632679
- added joint zed_right_camera_joint: type fixed, parent zed_camera_center, child zed_right_camera_frame, origin xyz=0 -0.0315 0 rpy=0 0 0
- added joint zed_right_camera_optical_joint: type fixed, parent zed_right_camera_frame, child zed_right_camera_optical_frame, origin xyz=0 0 0 rpy=-1.57079632679 0.0 -1.57079632679
